Commit message: Adding Skirt to R2 Model

File: urdf/robot_core.xacro (robot description, xacro)
@@ -81,5 +81,5 @@
     <gazebo reference="left_idler">
         <material>Gazebo/Blue</material>
-        <mu1>0</mu1>
+        <mu>0</mu>
         <mu2>0</mu2>
     </gazebo>
@@ -135,5 +135,5 @@
     <gazebo reference="right_idler">
         <material>Gazebo/Blue</material>
-        <mu1>0</mu1>
+        <mu>0</mu>
         <mu2>0</mu2>
     </gazebo>
@@ -193,4 +193,7 @@
         <axis xyz="0 -1 0" />
         <limit lower="-${radians(18)}" upper="${radians(2)}" velocity="100" effort="100" />
+        <xacro:unless value="$(arg sim_mode)">
+            <mimic joint="left_shoulder_joint" multiplier="0.5" offset="0" />
+        </xacro:unless>
     </joint>
     <link name="left_leg">
@@ -218,4 +221,7 @@
         <axis xyz="0 -1 0" />
         <limit lower="-${radians(18)}" upper="${radians(2)}" velocity="100" effort="100" />
+        <xacro:unless value="$(arg sim_mode)">
+            <mimic joint="right_shoulder_joint" multiplier="-0.5" offset="0" />
+        </xacro:unless>
     </joint>
     <link name="right_leg">
@@ -260,5 +266,6 @@
     <link name="shoulder">
     </link>
-    <xacro:property name="body_mass" value="1"/>
+    <!-- Let's make up a mass of 50kg -->
+    <xacro:property name="body_mass" value="50"/>
     <joint name="shoulder_link" type="fixed">
         <origin xyz="0 0 0" rpy="0 0 0" />
@@ -283,4 +290,32 @@
             <origin xyz="0 0 ${body_shoulder_offset - (body_height/2)}" rpy="0 0 0"/>
         </xacro:inertial_cylinder>
+    </link>
+    <!-- SKIRT -->
+    <xacro:property name="skirt_mass" value="1"/>
+    <xacro:property name="skirt_length" value="0.4616196"/>
+    <xacro:property name="skirt_width" value="0.3576574"/>
+    <xacro:property name="skirt_height" value="0.0635" />
+    <joint name="skirt_joint" type="fixed">
+        <parent link="body" />
+        <child link="skirt" />
+        <origin xyz="0 0 -${(body_height - body_shoulder_offset) + skirt_height}" rpy="${radians(90)} 0 ${radians(90)}" />
+    </joint>
+    <link name="skirt">
+        <visual>
+            <origin xyz="0 0 0" rpy="0 0 0" />
+            <geometry>
+                <mesh filename="package://r2_description/meshes/skirt.obj" />
+            </geometry>
+            <material name="white" />
+        </visual>
+        <collision>
+            <origin xyz="0 0 0" rpy="0 0 0" />
+            <geometry>
+                <mesh filename="package://r2_description/meshes/skirt.obj" />
+            </geometry>
+        </collision>
+        <xacro:inertial_box mass="${skirt_mass}" x="${skirt_width}" y="${skirt_height}" z="${skirt_length}">
+            <origin xyz="0 ${skirt_height/2} 0" rpy="0 0 0"/>
+        </xacro:inertial_box>
     </link>
     <!-- CENTER LEG -->
@@ -362,5 +397,5 @@
     <gazebo reference="center_front_idler">
         <material>Gazebo/Blue</material>
-        <mu1>0</mu1>
+        <mu>0</mu>
         <mu2>0</mu2>
     </gazebo>
@@ -389,5 +424,5 @@
     <gazebo reference="center_rear_idler">
         <material>Gazebo/Blue</material>
-        <mu1>0</mu1>
+        <mu>0</mu>
         <mu2>0</mu2>
     </gazebo>
