Commit message: Adding Utility Arm & LDP to URDF

File: urdf/properties.xacro (robot description, xacro)
@@ -43,3 +43,10 @@
   <xacro:property name="center_foot_depth" value="0.263525" />
   <xacro:property name="center_foot_height" value="0.1412748" />
+  <!-- Large Data Port -->
+  <xacro:property name="large_data_port_mass" value="0.5" />
+  <xacro:property name="large_data_port_width" value="0.127" />
+  <xacro:property name="large_data_port_length" value="0.127" />
+  <xacro:property name="large_data_port_height" value="${1.180 * 0.0254}" />
+  <!-- Top Utility Arm -->
+  <!-- Bottom Utility Arm -->
 </robot>

File: urdf/robot_core.xacro (robot description, xacro)
@@ -427,4 +427,59 @@
         <mu2>0</mu2>
     </gazebo>
+    <!-- Large Data Port -->
+    <joint name="large_data_port_joint" type="fixed">
+        <parent link="body" />
+        <child link="large_data_port" />
+        <origin xyz="0 0 ${body_shoulder_offset - large_data_port_height}" rpy="${radians(90)} 0 ${radians(90)}" />
+    </joint>
+    <link name="large_data_port">
+        <visual>
+            <origin xyz="0 0 0" rpy="0 0 0" />
+            <geometry>
+                <mesh filename="package://r2_description/meshes/large_data_port.obj" scale="0.001 0.001 0.001" />
+            </geometry>
+        </visual>
+        <collision>
+            <origin xyz="0 0 0" rpy="0 0 0" />
+            <geometry>
+                <mesh filename="package://r2_description/meshes/large_data_port.obj" scale="0.001 0.001 0.001" />
+            </geometry>
+        </collision>
+        <xacro:inertial_box mass="${large_data_port_mass}" x="${large_data_port_width}" y="${large_data_port_height}" z="${large_data_port_length}">
+            <origin xyz="0 ${large_data_port_height/2} 0" rpy="0 0 0"/>
+        </xacro:inertial_box>
+    </link>
+    <!-- Utility Arms -->
+    <xacro:macro name="utility_arm" params="name x y z angle_deg">
+        <xacro:property name="offsetX" value="${4.459 * 0.0254}" />
+        <xacro:property name="offsetY" value="${(1.375 / 2) * 0.0254}" />
+        <xacro:property name="offsetZ" value="${7.42 * 0.0254}" />
+        <joint name="${name}_joint" type="revolute">
+            <parent link="body" />
+            <child link="${name}" />
+            <origin xyz="${x} ${y} ${body_shoulder_offset - z}" rpy="${radians(90 + angle_deg)} 0 ${radians(90 + angle_deg)}" />
+            <axis xyz="0 1 0" />
+            <limit lower="0" upper="${radians(90)}" effort="100" velocity="100" />
+        </joint>
+        <link name="${name}">
+            <visual>
+                <origin xyz="${-offsetX} ${offsetY} ${-offsetZ}" rpy="0 0 ${radians(180)}" />
+                <geometry>
+                    <mesh filename="package://r2_description/meshes/utility_arm.obj" scale="0.001 0.001 0.001" />
+                </geometry>
+            </visual>
+            <collision>
+                <origin xyz="${-offsetX} ${offsetY} ${-offsetZ}" rpy="0 ${radians(180)} 0" />
+                <geometry>
+                    <mesh filename="package://r2_description/meshes/utility_arm.obj" scale="0.001 0.001 0.001" />
+                </geometry>
+            </collision>
+            <xacro:inertial_sphere mass="0.01" radius="0.01">
+                <origin xyz="0 0 0" rpy="0 0 0"/>
+            </xacro:inertial_sphere>
+        </link>
+    </xacro:macro>
+    <xacro:utility_arm name="upper_utility_arm" x="${7.42 * 0.0254}" y="${4.459 * 0.0254}" z="${((3.476-1.181) / 2 + 1.181) * 0.0254 - 0.002}" angle_deg="0" />
+    <xacro:utility_arm name="lower_utility_arm" x="${7.42 * 0.0254}" y="-${4.459 * 0.0254}" z="${((5.888-3.536) / 2 + 3.536) * 0.0254 - 0.002}" angle_deg="180" />
     <!-- DOME -->
     <joint name="dome_joint" type="continuous">
