Commit message: Adding a "mostly" working PP1 to demonstrate how to handle angles. Next we'll work on generating at least a properties file with the locations & angles available for import.

File: urdf/dome.xacro (robot description, xacro)
@@ -16,12 +16,15 @@
         </xacro:inertial_sphere>
     </link>
-    <joint name="pp1_joint" type="continuous">
+    <xacro:property name="pp1_angle" value="${radians(150)}" />
+    <joint name="pp1_joint" type="revolute">
         <parent link="dome" />
         <child link="pp1" />
-        <origin xyz="-0.114748 0.225099 0.06625" rpy="0 0 0" />
-        <axis xyz="1 0 0" />
+        <origin xyz="-0.114748 0.225099 0.06625" rpy="0 ${sin(pp1_angle)} 0" />
+        <axis xyz="0 0 1" />
+        <limit lower="0" upper="${radians(90)}" effort="100" velocity="100" />
     </joint>
     <link name="pp1">
         <visual>
+            <origin xyz="0 0 0" rpy="0 ${-sin(pp1_angle)} 0" />
             <geometry>
                 <mesh filename="package://r2_description/meshes/dome/PP1.obj" scale="0.01 0.01 0.01" />
@@ -29,4 +32,5 @@
         </visual>
         <collision>
+            <origin xyz="0 0 0" rpy="0 ${-sin(pp1_angle)} 0" />
             <geometry>
                 <mesh filename="package://r2_description/meshes/dome/PP1.obj" scale="0.01 0.01 0.01" />

Commit message: Updates to add the pie panels

File: urdf/dome.xacro (robot description, xacro)
@@ -1,4 +1,34 @@
 <?xml version="1.0"?>
 <robot xmlns:xacro="http://www.ros.org/wiki/xacro" >
+    <xacro:include filename="../meshes/dome/dome_constants.xacro"/>
+    <!-- R is Red Axis, P is Green Axis, Y is Blue Axis -->
+    <!---->
+    <xacro:macro name="pie_panel" params="name x y z angle_deg">
+        <xacro:property name="rot" value="${radians(90 - angle_deg)}" />
+        <joint name="${name}_joint" type="revolute">
+            <parent link="dome" />
+            <child link="${name}" />
+            <origin xyz="${x} ${y} ${z}" rpy="0 ${rot} 0" />
+            <axis xyz="1 0 0" />
+            <limit lower="0" upper="${radians(90)}" effort="100" velocity="100" />
+        </joint>
+        <link name="${name}">
+            <visual>
+                <origin xyz="0 0 0" rpy="0 ${-rot} 0" />
+                <geometry>
+                    <mesh filename="package://r2_description/meshes/dome/${name.upper()}.obj" scale="0.01 0.01 0.01" />
+                </geometry>
+            </visual>
+            <collision>
+                <origin xyz="0 0 0" rpy="0 ${-rot} 0" />
+                <geometry>
+                    <mesh filename="package://r2_description/meshes/dome/${name.upper()}.obj" scale="0.01 0.01 0.01" />
+                </geometry>
+            </collision>
+            <xacro:inertial_sphere mass="0.01" radius="0.01">
+                <origin xyz="0 0 0" rpy="0 0 0"/>
+            </xacro:inertial_sphere>
+        </link>
+    </xacro:macro>
     <link name="dome">
         <visual>
@@ -16,28 +46,8 @@
         </xacro:inertial_sphere>
     </link>
-    <xacro:property name="pp1_angle" value="${radians(150)}" />
-    <joint name="pp1_joint" type="revolute">
-        <parent link="dome" />
-        <child link="pp1" />
-        <origin xyz="-0.114748 0.225099 0.06625" rpy="0 ${sin(pp1_angle)} 0" />
-        <axis xyz="0 0 1" />
-        <limit lower="0" upper="${radians(90)}" effort="100" velocity="100" />
-    </joint>
-    <link name="pp1">
-        <visual>
-            <origin xyz="0 0 0" rpy="0 ${-sin(pp1_angle)} 0" />
-            <geometry>
-                <mesh filename="package://r2_description/meshes/dome/PP1.obj" scale="0.01 0.01 0.01" />
-            </geometry>
-        </visual>
-        <collision>
-            <origin xyz="0 0 0" rpy="0 ${-sin(pp1_angle)} 0" />
-            <geometry>
-                <mesh filename="package://r2_description/meshes/dome/PP1.obj" scale="0.01 0.01 0.01" />
-            </geometry>
-        </collision>
-        <xacro:inertial_sphere mass="1" radius="${dome_radius}">
-            <origin xyz="0 0 0" rpy="0 0 0"/>
-        </xacro:inertial_sphere>
-    </link>
+    <xacro:pie_panel name="pp1" x="${pp1_x}" y="${pp1_y}" z="${pp1_z}" angle_deg="${pp1_angle_deg}" />
+    <xacro:pie_panel name="pp2" x="${pp2_x}" y="${pp2_y}" z="${pp2_z}" angle_deg="${pp2_angle_deg}" />
+    <xacro:pie_panel name="pp4" x="${pp4_x}" y="${pp4_y}" z="${pp4_z}" angle_deg="${pp4_angle_deg}" />
+    <xacro:pie_panel name="pp5" x="${pp5_x}" y="${pp5_y}" z="${pp5_z}" angle_deg="${pp5_angle_deg}" />
+    <xacro:pie_panel name="pp6" x="${pp6_x}" y="${pp6_y}" z="${pp6_z}" angle_deg="${pp6_angle_deg}" />
 </robot>

Commit message: Add lower panels to dome. Inertia details still need to be implemented.

File: urdf/dome.xacro (robot description, xacro)
@@ -51,3 +51,39 @@
     <xacro:pie_panel name="pp5" x="${pp5_x}" y="${pp5_y}" z="${pp5_z}" angle_deg="${pp5_angle_deg}" />
     <xacro:pie_panel name="pp6" x="${pp6_x}" y="${pp6_y}" z="${pp6_z}" angle_deg="${pp6_angle_deg}" />
+    <!-- Lower Panels -->
+    <xacro:macro name="lower_panel" params="name x y z angle_deg">
+        <xacro:property name="rot" value="${radians(90 - angle_deg)}" />
+        <joint name="${name}_joint" type="revolute">
+            <parent link="dome" />
+            <child link="${name}" />
+            <origin xyz="${x} ${y} ${z}" rpy="0 ${rot} 0" />
+            <axis xyz="-1 0 0" />
+            <limit lower="0" upper="${radians(90)}" effort="100" velocity="100" />
+        </joint>
+        <link name="${name}">
+            <visual>
+                <origin xyz="0 0 0" rpy="0 ${-rot} 0" />
+                <geometry>
+                    <mesh filename="package://r2_description/meshes/dome/${name.upper()}.obj" scale="0.01 0.01 0.01" />
+                </geometry>
+            </visual>
+            <collision>
+                <origin xyz="0 0 0" rpy="0 ${-rot} 0" />
+                <geometry>
+                    <mesh filename="package://r2_description/meshes/dome/${name.upper()}.obj" scale="0.01 0.01 0.01" />
+                </geometry>
+            </collision>
+            <xacro:inertial_sphere mass="0.01" radius="0.01">
+                <origin xyz="0 0 0" rpy="0 0 0"/>
+            </xacro:inertial_sphere>
+        </link>
+    </xacro:macro>
+    <xacro:lower_panel name="p1" x="${p1_x}" y="${p1_y}" z="${p1_z}" angle_deg="${p1_angle_deg}" />
+    <xacro:lower_panel name="p2" x="${p2_x}" y="${p2_y}" z="${p2_z}" angle_deg="${p2_angle_deg}" />
+    <xacro:lower_panel name="p3" x="${p3_x}" y="${p3_y}" z="${p3_z}" angle_deg="${p3_angle_deg}" />
+    <xacro:lower_panel name="p4" x="${p4_x}" y="${p4_y}" z="${p4_z}" angle_deg="${p4_angle_deg}" />
+    <xacro:lower_panel name="p7" x="${p7_x}" y="${p7_y}" z="${p7_z}" angle_deg="${p7_angle_deg}" />
+    <xacro:lower_panel name="p10" x="${p10_x}" y="${p10_y}" z="${p10_z}" angle_deg="${p10_angle_deg}" />
+    <xacro:lower_panel name="p11" x="${p11_x}" y="${p11_y}" z="${p11_z}" angle_deg="${p11_angle_deg}" />
+    <xacro:lower_panel name="p13" x="${p13_x}" y="${p13_y}" z="${p13_z}" angle_deg="${p13_angle_deg}" />
 </robot>

Commit message: Updates to add body opening panels

File: urdf/dome.xacro (robot description, xacro)
@@ -31,4 +31,10 @@
         </link>
     </xacro:macro>
+    <joint name="dome_joint" type="continuous">
+        <parent link="body" />
+        <child link="dome" />
+        <origin xyz="0 0 ${dome_offset}" rpy="${radians(90)} 0 ${radians(180)}" />
+        <axis xyz="0 -1 0" />
+    </joint>
     <link name="dome">
         <visual>

File: urdf/robot_core.xacro (robot description, xacro)
@@ -273,22 +273,4 @@
         <child link="body" />
     </joint>
-    <link name="body">
-        <visual>
-            <origin xyz="0 0 ${body_shoulder_offset}" rpy="${radians(90)} 0 ${radians(90)}" />
-            <geometry>
-                <!-- Exported in meters -->
-                <mesh filename="package://r2_description/meshes/frame.obj" scale="1 1 1" />
-            </geometry>
-        </visual>
-        <collision>
-            <origin xyz="0 0 ${body_shoulder_offset}" rpy="${radians(90)} 0 ${radians(90)}" />
-            <geometry>
-                <mesh filename="package://r2_description/meshes/frame.obj" scale="1 1 1" />
-            </geometry>
-        </collision>
-        <xacro:inertial_cylinder mass="${body_mass}" length="${body_height}" radius="${body_radius}">
-            <origin xyz="0 0 ${body_shoulder_offset - (body_height/2)}" rpy="0 0 0"/>
-        </xacro:inertial_cylinder>
-    </link>
     <!-- SKIRT -->
     <xacro:property name="skirt_mass" value="1"/>
@@ -427,83 +409,6 @@
         <mu2>0</mu2>
     </gazebo>
-    <!-- Large Data Port -->
-    <joint name="large_data_port_joint" type="fixed">
-        <parent link="body" />
-        <child link="large_data_port" />
-        <origin xyz="0 0 ${body_shoulder_offset - large_data_port_height}" rpy="${radians(90)} 0 ${radians(90)}" />
-    </joint>
-    <link name="large_data_port">
-        <visual>
-            <origin xyz="0 0 0" rpy="0 0 0" />
-            <geometry>
-                <mesh filename="package://r2_description/meshes/large_data_port.obj" scale="0.001 0.001 0.001" />
-            </geometry>
-        </visual>
-        <collision>
-            <origin xyz="0 0 0" rpy="0 0 0" />
-            <geometry>
-                <mesh filename="package://r2_description/meshes/large_data_port.obj" scale="0.001 0.001 0.001" />
-            </geometry>
-        </collision>
-        <xacro:inertial_box mass="${large_data_port_mass}" x="${large_data_port_width}" y="${large_data_port_height}" z="${large_data_port_length}">
-            <origin xyz="0 ${large_data_port_height/2} 0" rpy="0 0 0"/>
-        </xacro:inertial_box>
-    </link>
-    <!-- Utility Arms -->
-    <xacro:macro name="utility_arm" params="name x y z angle_deg">
-        <xacro:property name="offsetX" value="${4.459 * 0.0254}" />
-        <xacro:property name="offsetY" value="${(1.375 / 2) * 0.0254}" />
-        <xacro:property name="offsetZ" value="${7.42 * 0.0254}" />
-        <joint name="${name}_joint" type="revolute">
-            <parent link="body" />
-            <child link="${name}" />
-            <origin xyz="${x} ${y} ${body_shoulder_offset - z}" rpy="${radians(90 + angle_deg)} 0 ${radians(90 + angle_deg)}" />
-            <axis xyz="0 1 0" />
-            <limit lower="0" upper="${radians(90)}" effort="100" velocity="100" />
-        </joint>
-        <link name="${name}">
-            <visual>
-                <origin xyz="${-offsetX} ${offsetY} ${-offsetZ}" rpy="0 0 ${radians(180)}" />
-                <geometry>
-                    <mesh filename="package://r2_description/meshes/utility_arm.obj" scale="0.001 0.001 0.001" />
-                </geometry>
-            </visual>
-            <collision>
-                <origin xyz="${-offsetX} ${offsetY} ${-offsetZ}" rpy="0 ${radians(180)} 0" />
-                <geometry>
-                    <mesh filename="package://r2_description/meshes/utility_arm.obj" scale="0.001 0.001 0.001" />
-                </geometry>
-            </collision>
-            <xacro:inertial_sphere mass="0.01" radius="0.01">
-                <origin xyz="0 0 0" rpy="0 0 0"/>
-            </xacro:inertial_sphere>
-        </link>
-    </xacro:macro>
-    <xacro:utility_arm name="upper_utility_arm" x="${7.42 * 0.0254}" y="${4.459 * 0.0254}" z="${((3.476-1.181) / 2 + 1.181) * 0.0254 - 0.002}" angle_deg="0" />
-    <xacro:utility_arm name="lower_utility_arm" x="${7.42 * 0.0254}" y="-${4.459 * 0.0254}" z="${((5.888-3.536) / 2 + 3.536) * 0.0254 - 0.002}" angle_deg="180" />
+    <xacro:include filename="body.xacro" />
     <!-- DOME -->
-    <joint name="dome_joint" type="continuous">
-        <parent link="body" />
-        <child link="dome" />
-        <origin xyz="0 0 ${dome_offset}" rpy="${radians(90)} 0 ${radians(180)}" />
-        <axis xyz="0 -1 0" />
-    </joint>
     <xacro:include filename="dome.xacro" />
-    <!--
-    <link name="dome">
-        <visual>
-            <geometry>
-                <mesh filename="package://r2_description/meshes/dome.obj" />
-            </geometry>
-        </visual>
-        <collision>
-            <geometry>
-                <mesh filename="package://r2_description/meshes/dome.obj" />
-            </geometry>
-        </collision>
-        <xacro:inertial_sphere mass="1" radius="${dome_radius}">
-            <origin xyz="0 0 0" rpy="0 0 0"/>
-        </xacro:inertial_sphere>
-    </link>
-    -->
 </robot>
