Commit message: urdf: mark servo-driven joints and give them display names
The dome panel needs to know which joints are driven by a servo and what to
call them on screen, and URDF has no way to say either. Adds a vendor
extension under https://astromech.co/urdf/1.0: one optional child of <joint>
whose presence means "this joint is driven by a servo".

    <astromech:servo display="PIE PANEL 1" />

Only `display` is defined at 1.0. Where the servo actually lives is
deliberately not in the schema -- a controller knows its own channels, so a
tagged joint it has no channel for is by definition driven by something else.

All 22 come from four macros, so this is four macro edits plus a name per call
site: pie_panel (5), lower_panel (8), body_panel (7), utility_arm (2). The
ankles, shoulder and center_foot are revolute too but are left untagged; tag
them if they turn out to be servos.

Verified by expanding robot_core.xacro locally: xacro preserves the
xmlns:astromech declaration on the output root (it strips only its own), and
all 22 elements survive into the flattened URDF, which is what
robot_state_publisher republishes verbatim.

Co-Authored-By: Claude Opus 5 <noreply@anthropic.com>

File: urdf/body.xacro (robot description, xacro)
@@ -1,6 +1,7 @@
 <?xml version="1.0"?>
-<robot xmlns:xacro="http://www.ros.org/wiki/xacro" >
+<robot xmlns:xacro="http://www.ros.org/wiki/xacro"
+       xmlns:astromech="https://astromech.co/urdf/1.0" >
     <xacro:include filename="../meshes/body/skin_constants.xacro" />
-    <xacro:macro name="body_panel" params="name x y z angle_deg">
+    <xacro:macro name="body_panel" params="name display x y z angle_deg">
         <xacro:property name="rot" value="${radians(angle_deg)}" />
         <xacro:property name="rotation_mult" value="-1" />
@@ -14,4 +15,5 @@
             <axis xyz="0 0 ${rotation_mult}" />
             <limit lower="0" upper="${radians(90)}" effort="100" velocity="100" />
+            <astromech:servo display="${display}" />
         </joint>
         <link name="${name}">
@@ -52,11 +54,11 @@
         </xacro:inertial_cylinder>
     </link>
-    <xacro:body_panel name="bf1" x="${bf1_z}" y="${bf1_x}" z="${bf1_y}" angle_deg="${bf1_angle_deg}" />
-    <xacro:body_panel name="bf2" x="${bf2_z}" y="${bf2_x}" z="${bf2_y}" angle_deg="${bf2_angle_deg}" />
-    <xacro:body_panel name="bf3" x="${bf3_z}" y="${bf3_x}" z="${bf3_y}" angle_deg="${bf3_angle_deg}" />
-    <xacro:body_panel name="bf4" x="${bf4_z}" y="${bf4_x}" z="${bf4_y}" angle_deg="${bf4_angle_deg}" />
-    <xacro:body_panel name="bf5" x="${bf5_z}" y="${bf5_x}" z="${bf5_y}" angle_deg="${bf5_angle_deg}" />
-    <xacro:body_panel name="br1" x="${br1_z}" y="${br1_x}" z="${br1_y}" angle_deg="${br1_angle_deg}" />
-    <xacro:body_panel name="br6" x="${br6_z}" y="${br6_x}" z="${br6_y}" angle_deg="${br6_angle_deg}" />
+    <xacro:body_panel name="bf1" display="BODY FRONT 1" x="${bf1_z}" y="${bf1_x}" z="${bf1_y}" angle_deg="${bf1_angle_deg}" />
+    <xacro:body_panel name="bf2" display="BODY FRONT 2" x="${bf2_z}" y="${bf2_x}" z="${bf2_y}" angle_deg="${bf2_angle_deg}" />
+    <xacro:body_panel name="bf3" display="BODY FRONT 3" x="${bf3_z}" y="${bf3_x}" z="${bf3_y}" angle_deg="${bf3_angle_deg}" />
+    <xacro:body_panel name="bf4" display="BODY FRONT 4" x="${bf4_z}" y="${bf4_x}" z="${bf4_y}" angle_deg="${bf4_angle_deg}" />
+    <xacro:body_panel name="bf5" display="BODY FRONT 5" x="${bf5_z}" y="${bf5_x}" z="${bf5_y}" angle_deg="${bf5_angle_deg}" />
+    <xacro:body_panel name="br1" display="BODY REAR 1" x="${br1_z}" y="${br1_x}" z="${br1_y}" angle_deg="${br1_angle_deg}" />
+    <xacro:body_panel name="br6" display="BODY REAR 6" x="${br6_z}" y="${br6_x}" z="${br6_y}" angle_deg="${br6_angle_deg}" />
     <!-- Large Data Port -->
     <joint name="large_data_port_joint" type="fixed">
@@ -83,5 +85,5 @@
     </link>
     <!-- Utility Arms -->
-    <xacro:macro name="utility_arm" params="name x y z angle_deg">
+    <xacro:macro name="utility_arm" params="name display x y z angle_deg">
         <xacro:property name="offsetX" value="${4.459 * 0.0254}" />
         <xacro:property name="offsetY" value="${(1.375 / 2) * 0.0254}" />
@@ -93,4 +95,5 @@
             <axis xyz="0 1 0" />
             <limit lower="0" upper="${radians(90)}" effort="100" velocity="100" />
+            <astromech:servo display="${display}" />
         </joint>
         <link name="${name}">
@@ -112,5 +115,5 @@
         </link>
     </xacro:macro>
-    <xacro:utility_arm name="upper_utility_arm" x="${7.42 * 0.0254}" y="${4.459 * 0.0254}" z="${((3.476-1.181) / 2 + 1.181) * 0.0254 - 0.002}" angle_deg="0" />
-    <xacro:utility_arm name="lower_utility_arm" x="${7.42 * 0.0254}" y="-${4.459 * 0.0254}" z="${((5.888-3.536) / 2 + 3.536) * 0.0254 - 0.002}" angle_deg="180" />
+    <xacro:utility_arm name="upper_utility_arm" display="UPPER UTILITY ARM" x="${7.42 * 0.0254}" y="${4.459 * 0.0254}" z="${((3.476-1.181) / 2 + 1.181) * 0.0254 - 0.002}" angle_deg="0" />
+    <xacro:utility_arm name="lower_utility_arm" display="LOWER UTILITY ARM" x="${7.42 * 0.0254}" y="-${4.459 * 0.0254}" z="${((5.888-3.536) / 2 + 3.536) * 0.0254 - 0.002}" angle_deg="180" />
 </robot>

File: urdf/dome.xacro (robot description, xacro)
@@ -1,8 +1,9 @@
 <?xml version="1.0"?>
-<robot xmlns:xacro="http://www.ros.org/wiki/xacro" >
+<robot xmlns:xacro="http://www.ros.org/wiki/xacro"
+       xmlns:astromech="https://astromech.co/urdf/1.0" >
     <xacro:include filename="../meshes/dome/dome_constants.xacro"/>
     <!-- R is Red Axis, P is Green Axis, Y is Blue Axis -->
     <!---->
-    <xacro:macro name="pie_panel" params="name x y z angle_deg">
+    <xacro:macro name="pie_panel" params="name display x y z angle_deg">
         <xacro:property name="rot" value="${radians(90 - angle_deg)}" />
         <joint name="${name}_joint" type="revolute">
@@ -12,4 +13,5 @@
             <axis xyz="1 0 0" />
             <limit lower="0" upper="${radians(90)}" effort="100" velocity="100" />
+            <astromech:servo display="${display}" />
         </joint>
         <link name="${name}">
@@ -52,11 +54,11 @@
         </xacro:inertial_sphere>
     </link>
-    <xacro:pie_panel name="pp1" x="${pp1_x}" y="${pp1_y}" z="${pp1_z}" angle_deg="${pp1_angle_deg}" />
-    <xacro:pie_panel name="pp2" x="${pp2_x}" y="${pp2_y}" z="${pp2_z}" angle_deg="${pp2_angle_deg}" />
-    <xacro:pie_panel name="pp4" x="${pp4_x}" y="${pp4_y}" z="${pp4_z}" angle_deg="${pp4_angle_deg}" />
-    <xacro:pie_panel name="pp5" x="${pp5_x}" y="${pp5_y}" z="${pp5_z}" angle_deg="${pp5_angle_deg}" />
-    <xacro:pie_panel name="pp6" x="${pp6_x}" y="${pp6_y}" z="${pp6_z}" angle_deg="${pp6_angle_deg}" />
+    <xacro:pie_panel name="pp1" display="PIE PANEL 1" x="${pp1_x}" y="${pp1_y}" z="${pp1_z}" angle_deg="${pp1_angle_deg}" />
+    <xacro:pie_panel name="pp2" display="PIE PANEL 2" x="${pp2_x}" y="${pp2_y}" z="${pp2_z}" angle_deg="${pp2_angle_deg}" />
+    <xacro:pie_panel name="pp4" display="PIE PANEL 4" x="${pp4_x}" y="${pp4_y}" z="${pp4_z}" angle_deg="${pp4_angle_deg}" />
+    <xacro:pie_panel name="pp5" display="PIE PANEL 5" x="${pp5_x}" y="${pp5_y}" z="${pp5_z}" angle_deg="${pp5_angle_deg}" />
+    <xacro:pie_panel name="pp6" display="PIE PANEL 6" x="${pp6_x}" y="${pp6_y}" z="${pp6_z}" angle_deg="${pp6_angle_deg}" />
     <!-- Lower Panels -->
-    <xacro:macro name="lower_panel" params="name x y z angle_deg">
+    <xacro:macro name="lower_panel" params="name display x y z angle_deg">
         <xacro:property name="rot" value="${radians(90 - angle_deg)}" />
         <joint name="${name}_joint" type="revolute">
@@ -66,4 +68,5 @@
             <axis xyz="-1 0 0" />
             <limit lower="0" upper="${radians(90)}" effort="100" velocity="100" />
+            <astromech:servo display="${display}" />
         </joint>
         <link name="${name}">
@@ -85,11 +88,11 @@
         </link>
     </xacro:macro>
-    <xacro:lower_panel name="p1" x="${p1_x}" y="${p1_y}" z="${p1_z}" angle_deg="${p1_angle_deg}" />
-    <xacro:lower_panel name="p2" x="${p2_x}" y="${p2_y}" z="${p2_z}" angle_deg="${p2_angle_deg}" />
-    <xacro:lower_panel name="p3" x="${p3_x}" y="${p3_y}" z="${p3_z}" angle_deg="${p3_angle_deg}" />
-    <xacro:lower_panel name="p4" x="${p4_x}" y="${p4_y}" z="${p4_z}" angle_deg="${p4_angle_deg}" />
-    <xacro:lower_panel name="p7" x="${p7_x}" y="${p7_y}" z="${p7_z}" angle_deg="${p7_angle_deg}" />
-    <xacro:lower_panel name="p10" x="${p10_x}" y="${p10_y}" z="${p10_z}" angle_deg="${p10_angle_deg}" />
-    <xacro:lower_panel name="p11" x="${p11_x}" y="${p11_y}" z="${p11_z}" angle_deg="${p11_angle_deg}" />
-    <xacro:lower_panel name="p13" x="${p13_x}" y="${p13_y}" z="${p13_z}" angle_deg="${p13_angle_deg}" />
+    <xacro:lower_panel name="p1" display="LOWER PANEL 1" x="${p1_x}" y="${p1_y}" z="${p1_z}" angle_deg="${p1_angle_deg}" />
+    <xacro:lower_panel name="p2" display="LOWER PANEL 2" x="${p2_x}" y="${p2_y}" z="${p2_z}" angle_deg="${p2_angle_deg}" />
+    <xacro:lower_panel name="p3" display="LOWER PANEL 3" x="${p3_x}" y="${p3_y}" z="${p3_z}" angle_deg="${p3_angle_deg}" />
+    <xacro:lower_panel name="p4" display="LOWER PANEL 4" x="${p4_x}" y="${p4_y}" z="${p4_z}" angle_deg="${p4_angle_deg}" />
+    <xacro:lower_panel name="p7" display="LOWER PANEL 7" x="${p7_x}" y="${p7_y}" z="${p7_z}" angle_deg="${p7_angle_deg}" />
+    <xacro:lower_panel name="p10" display="LOWER PANEL 10" x="${p10_x}" y="${p10_y}" z="${p10_z}" angle_deg="${p10_angle_deg}" />
+    <xacro:lower_panel name="p11" display="LOWER PANEL 11" x="${p11_x}" y="${p11_y}" z="${p11_z}" angle_deg="${p11_angle_deg}" />
+    <xacro:lower_panel name="p13" display="LOWER PANEL 13" x="${p13_x}" y="${p13_y}" z="${p13_z}" angle_deg="${p13_angle_deg}" />
 </robot>
